Commit message: robot.urdf: add a new link to the robot

File: hospital_robot/urdf/robot.urdf (robot description, URDF)
Before this commit: robot hospital_robot, 2 links, 1 joints
Links:
- link base_link: mass None -> 5.0; geometry collision box size=${length} ${breadth} ${height}; visual box size=${length} ${breadth} ${height}
- link lidar_link: mass None -> 0.1; geometry collision cylinder length=0.05 radius=0.05; visual cylinder length=0.05 radius=0.05
Joints:
- joint lidar_joint: origin xyz=0 0 0.15 rpy=0 0 0 -> xyz=0 0 ${height} rpy=0 0 0

Commit message: final urdf file commit

File: hospital_robot/urdf/robot.urdf (robot description, URDF)
Before this commit: robot my_robot, 2 links, 1 joints
Links:
- added link dummy_link, mass 0.01; collision sphere radius=0.02; visual sphere radius=0.02
- added link dummy_root_link
- added link lidar_box_link, mass 0.5; collision box size=0.12 0.30 0.1; visual box size=0.12 0.30 0.1
- added link lock_link, mass 0.1; collision box size=0.05 0.02 0.05; visual box size=0.05 0.02 0.05
- added link wheel_1, mass 0.5; collision cylinder length=0.02 radius=0.031; visual cylinder length=0.02 radius=0.031
- added link wheel_2, mass 0.5; collision cylinder length=0.02 radius=0.031; visual cylinder length=0.02 radius=0.031
- added link wheel_3, mass 0.5; collision cylinder length=0.02 radius=0.031; visual cylinder length=0.02 radius=0.031
- added link wheel_4, mass 0.5; collision cylinder length=0.02 radius=0.031; visual cylinder length=0.02 radius=0.031
- link base_link: geometry collision box size=0.32 0.30 0.40; visual box size=0.32 0.30 0.40
- link lidar_link: mass 0.1 -> 0.2; geometry collision cylinder length=0.045 radius=0.0375; visual cylinder length=0.045 radius=0.0375
Joints:
- added joint dummy_joint: type fixed, parent base_link, child dummy_link, origin xyz=0.0 0.0 0.25 rpy=0 0 0
- added joint dummy_root_joint: type fixed, parent dummy_root_link, child base_link, origin xyz=0 0 0 rpy=0 0 0
- added joint lidar_box_joint: type fixed, parent base_link, child lidar_box_link, origin xyz=0 0 0.4 rpy=0 0 0
- added joint lock_joint: type fixed, parent base_link, child lock_link, origin xyz=0.15 0.12 0.25 rpy=0 0 0
- added joint wheel_1_joint: type continuous, parent base_link, child wheel_1, origin xyz=0.15 0.15 -0.02 rpy=0 0 0, axis 0 1 0
- added joint wheel_2_joint: type continuous, parent base_link, child wheel_2, origin xyz=0.15 -0.15 -0.02 rpy=0 0 0, axis 0 1 0
- added joint wheel_3_joint: type continuous, parent base_link, child wheel_3, origin xyz=-0.15 0.15 -0.02 rpy=0 0 0, axis 0 1 0
- added joint wheel_4_joint: type continuous, parent base_link, child wheel_4, origin xyz=-0.15 -0.15 -0.02 rpy=0 0 0, axis 0 1 0
- joint lidar_joint: origin xyz=0 0 ${height} rpy=0 0 0 -> xyz=-0.1 0 0.05 rpy=0 0 0; parent base_link -> lidar_box_link

Commit message: Update robot.urdf

File: hospital_robot/urdf/robot.urdf (robot description, URDF)
Before this commit: robot my_robot, 10 links, 9 joints
Links:
- link base_link: mass 5.0 -> 0.5
- link lidar_box_link: mass 0.5 -> 0.09
- link lock_link: mass 0.1 -> 0.01
- link wheel_1: mass 0.5 -> 0.01
- link wheel_2: mass 0.5 -> 0.01
- link wheel_3: mass 0.5 -> 0.01
- link wheel_4: mass 0.5 -> 0.01

Commit message: Update robot.urdf

File: hospital_robot/urdf/robot.urdf (robot description, URDF)
Before this commit: robot my_robot, 10 links, 9 joints
Links:
- link base_link: mass 0.5 -> 5.0
- link lidar_box_link: mass 0.09 -> 0.5
- link lock_link: mass 0.01 -> 0.1
- link wheel_1: mass 0.01 -> 0.5
- link wheel_2: mass 0.01 -> 0.5
- link wheel_3: mass 0.01 -> 0.5
- link wheel_4: mass 0.01 -> 0.5
